File: PCB/energy_metering.kicad_sch (KiCad schematic)
At the start: 86 parts, among them J2 Screw_Terminal_01x04, J3 Screw_Terminal_01x08, J4 Conn_02x06_Odd_Even, U5 ATM90E36A-AU-R, Y1 ABM8W-16.3840MHZ-4-B1U-T3

Commit message: added MD50 PDFs and oled 3d model
Other:
- note added: "Utilizar sensor de corrente SCT-013"
Changed lines of the file:
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@@
 	(generator_version "10.0")
 	(paper "A4")
+	(text "Utilizar sensor de corrente\nSCT-013"
+		(exclude_from_sim no)
+		(at 153.162 146.812 0)
+		(effects
+			(font
+				(size 2 2)
+				(thickness 0.254)
+				(bold yes)
+				(color 0 0 0 1)
+			)
+		)
+	)
 	(junction
 		(at 96.52 143.51)
@@
 		)
 	)
-	(embedded_fonts no)
 )

Commit message: edited the PCB layout
Parts:
- added TP12, TP14, TP28: TestPoint, TestPoint:TestPoint_Pad_D1.0mm, symbol Connector:TestPoint
Connections:
- net CF1: now also J4.6 (Pin_6); no longer J4.8 (Pin_8)
- net CF2: now also J4.3 (Pin_3); no longer J4.10 (Pin_10)
- net CF3: now also J4.7 (Pin_7); no longer J4.12 (Pin_12)
- net CF4: now also J4.4 (Pin_4); no longer J4.1 (Pin_1)
- net DMA: now also J4.2 (Pin_2); no longer J4.9 (Pin_9)
- net IRQ0: now also J4.1 (Pin_1); no longer J4.5 (Pin_5)
- net IRQ1: now also J4.5 (Pin_5); no longer J4.7 (Pin_7)
- net V1P: now also TP12.1
- net V2P: now also TP14.1
- net V3P: now also TP28.1
- net WARN: now also J4.8 (Pin_8); no longer J4.3 (Pin_3)
- net ZX0: now also J4.12 (Pin_12); no longer J4.2 (Pin_2)
- net ZX1: now also J4.9 (Pin_9); no longer J4.4 (Pin_4)
- net ZX2: now also J4.10 (Pin_10); no longer J4.6 (Pin_6)

Commit message: PCB routing and adjusts
Parts:
- renumbered C26 to C18, C39 to C19, C18 to C20, C19 to C21, C20 to C22, C21 to C23, C22 to C24, C23 to C25, C24 to C26, C37 to C27, C38 to C28, J2 to J7, J3 to J8, J4 to J9, R8 to R11, R9 to R12, R10 to R13, R11 to R14, R12 to R15, R13 to R16, R14 to R17, R15 to R18, R16 to R19, R17 to R20, R18 to R21, R19 to R22, R20 to R23, R21 to R24, R22 to R25, R23 to R26, R30 to R27, R31 to R28, R35 to R29, R36 to R30, R24 to R31, R25 to R32, R26 to R33, R27 to R34, R28 to R35, R29 to R36, R32 to R37, R33 to R38, R34 to R39, R37 to R40, R38 to R41, R39 to R42, R40 to R43, R41 to R44, R42 to R45, R44 to R46, R45 to R47, R47 to R48, R48 to R49, R43 to R50, R46 to R51, R64 to R52, R65 to R53, R49 to R54, R66 to R55, R67 to R56, R50 to R57, R51 to R58, TP7 to TP1, TP28 to TP10, TP25 to TP11, TP26 to TP12, TP17 to TP13, TP8 to TP2, TP9 to TP3, TP10 to TP4, TP11 to TP5, TP15 to TP6, TP16 to TP7, TP12 to TP8, TP14 to TP9
Other:
- moved on the sheet: R13, R14, R15, R18, R19, R20, R21, R22, R23, R24, R25, R26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

Commit message: altered the solder mask expansion and added pcb cutout under esp antenna
Parts:
- U5: footprint 1lib:48TQFP -> myLIB:48TQFP
Changed lines of the file:
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@@
 			)
 		)
-		(property "Footprint" "1lib:48TQFP"
+		(property "Footprint" "myLIB:48TQFP"
 			(at 190.5 87.63 0)
 			(hide yes)
