File: PCB/isolation.kicad_sch (KiCad schematic)
At the start: 43 parts, among them J5 Conn_01x03, U10 TPS22918DBV, U6 HLK-5M05, U7 B0303S-1WR3, U8 BQ24073RGT, U9 TLV75733PDRV

Commit message: PCB routing and adjusts
Parts:
- added TP21: TestPoint, TestPoint:TestPoint_Pad_D1.5mm, symbol Connector:TestPoint
- renumbered C25 to C29, C27 to C30, C28 to C31, C29 to C32, C30 to C33, C31 to C34, C32 to C35, C33 to C36, C34 to C37, C35 to C38, C36 to C39, D4 to D5, D5 to D6, D6 to D7, D7 to D8, J5 to J10, JP2 to JP1, R52 to R59, R53 to R60, R54 to R61, R55 to R62, R56 to R63, R57 to R64, R58 to R65, R59 to R66, R60 to R67, R61 to R68, R62 to R69, R63 to R70, TP18 to TP14, TP19 to TP15, TP24 to TP16, TP23 to TP17, TP22 to TP18, TP20 to TP19, TP21 to TP20
Connections:
- net GND: now also TP21.1

Commit message: altered the solder mask expansion and added pcb cutout under esp antenna
Parts:
- U7: footprint 1lib:B0303S-1WR3 -> myLIB:B0303S-1WR3
Changed lines of the file:
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@@
 			)
 		)
-		(property "Footprint" "1lib:B0303S-1WR3"
+		(property "Footprint" "myLIB:B0303S-1WR3"
 			(at 60.96 115.57 0)
 			(hide yes)
