File: PCB/isolation.kicad_sch (KiCad schematic)
At the start: 44 parts, among them J10 Conn_01x03, U10 TPS22918DBV, U6 HLK-5M05, U7 B0303S-1WR3, U8 BQ24073RGT, U9 TLV75733PDRV

Commit message: new readme, added .step models to pcb
Parts:
- F1: footprint 1lib:FuseHolder_5x20mm_P=22,5mm -> myLIB:FuseHolder_5x20mm_P=22,5mm
Changed lines of the file:
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@@
 			)
 		)
-		(property "Footprint" "1lib:FuseHolder_5x20mm_P=22,5mm"
+		(property "Footprint" "myLIB:FuseHolder_5x20mm_P=22,5mm"
 			(at 29.21 27.94 0)
 			(hide yes)
