File: PCB/digital.kicad_sch (KiCad schematic)
At the start: 24 parts, among them J1 Conn_01x06, U1 ESP32-S3, U2 PC817, U3 PC817, U4 ADuM1411

Commit message: addded oled screen and wifi led
Parts:
- added D8: LED_L3, LED_SMD:LED_0603_1608Metric, symbol Device:LED
- added R68, R69: 10k, Resistor_SMD:R_0603_1608Metric, symbol Device:R
- added R70: 1k, Resistor_SMD:R_0603_1608Metric, symbol Device:R
- added U11: (no value), myLIB:128x64OLED, symbol myLIB:OLED_I2C_128x64
Connections:
- net IO45 is gone; now on net PMC_1: U1.26 (IO45)
- net IO48 is gone; now on net PMC_0: U1.25 (IO48)
- net +3V3: now also R68.1, R69.1, U11.2 (VDD)
- net GND: now also D8.1 (K), U11.1 (GND)
- net PMC_0: no longer U1.5 (IO5)
- net PMC_1: no longer U1.6 (IO6)
- net IO40 renamed SDA
- net SDA: now also R68.2, U11.4 (SDA)
- net IO41 renamed SCL
- net SCL: now also R69.2, U11.3 (SCL)
- new net: D8.2 (A), R70.2
- new net IO5: U1.5 (IO5)
- new net LED_WIFI: R70.1, U1.6 (IO6)

Commit message: edited the PCB layout
Parts:
- removed U11: (no value), myLIB:128x64OLED, symbol myLIB:OLED_I2C_128x64
- added J10, J7, J8, J9: Conn_01x02, Connector_PinHeader_2.54mm:PinHeader_1x02_P2.54mm_Vertical, symbol Connector_Generic:Conn_01x02
- added J6: Conn_01x04, Connector_PinHeader_2.54mm:PinHeader_1x04_P2.54mm_Vertical, symbol Connector_Generic:Conn_01x04
Connections:
- net +3V3: now also J6.2 (Pin_2)
- net GND: now also J10.2 (Pin_2), J6.1 (Pin_1), J7.2 (Pin_2), J8.2 (Pin_2), J9.2 (Pin_2)
- net PMC_0: now also U1.26 (IO45); no longer U1.25 (IO48)
- net PMC_1: now also U1.25 (IO48); no longer U1.26 (IO45)
- net SCL: now also R68.2, J6.3 (Pin_3); no longer R69.2
- net SDA: now also R69.2, J6.4 (Pin_4); no longer R68.2
- net at D2.2 (A), R2.2: now also J8.1 (Pin_1)
- net at D3.2 (A), R3.2: now also J7.1 (Pin_1)
- net at D1.2 (A), R1.2: now also J9.1 (Pin_1)
- net at D8.2 (A), R70.2: now also J10.1 (Pin_1)
Other:
- note added: "OLED I2C"
- moved on the sheet: C1, C2, C3, C4, C5, D1, D2, D3, D8, H1, H2, H3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

Commit message: PCB routing and adjusts
Parts:
- renumbered D8 to D4, J9 to J1, J8 to J2, J6 to J3, J1 to J4, J7 to J5, J10 to J6, R7 to R10, R68 to R4, R69 to R5, R70 to R6, R4 to R7, R5 to R8, R6 to R9

Commit message: altered the solder mask expansion and added pcb cutout under esp antenna
Parts:
- U2, U3: footprint 1lib:SOIC-4_6.5x4.6_P2.54mm -> myLIB:SOIC-4_6.5x4.6_P2.54mm
Changed lines of the file:
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@@
 			)
 		)
-		(property "Footprint" "1lib:SOIC-4_6.5x4.6_P2.54mm"
+		(property "Footprint" "myLIB:SOIC-4_6.5x4.6_P2.54mm"
 			(at 219.71 39.37 0)
 			(hide yes)
@@
 			)
 		)
-		(property "Footprint" "1lib:SOIC-4_6.5x4.6_P2.54mm"
+		(property "Footprint" "myLIB:SOIC-4_6.5x4.6_P2.54mm"
 			(at 219.71 67.31 0)
 			(hide yes)

Commit message: added pullup resistor on EN pin + cap to gnd on the same pin
Parts:
- added C40: 100n/16V, Capacitor_SMD:C_0603_1608Metric, symbol Device:C
- added R71: 10k, Resistor_SMD:R_0603_1608Metric, symbol Device:R
Connections:
- net +3V3: now also R71.1
- net EN: now also C40.1, R71.2
- net GND: now also C40.2
